Commit message: new robot chassis and testing launch files

File: urdf/macros.xacro (robot description, xacro)
@@ -42,7 +42,9 @@
   <!-- geometry macros -->
   <xacro:macro name="chassis_geometry">
-    <origin xyz="0.46 -0.135 -0.180" rpy="1.57 0 3.14" />
-    <geometry>
-      <mesh filename="package://spring_2020_virtual_class/urdf/meshes/chassis.stl" scale="0.000990 0.0009375 0.0009375"/>
+    <!-- <origin xyz="0.46 -0.135 -0.180" rpy="1.57 0 3.14" /> -->
+    <origin rpy="-1.5708 0 3.1416" xyz="0.175 0.35 0.07"/>
+    <geometry>
+      <mesh filename="package://f1tenth-sim/urdf/meshes/chassis.STL" scale="0.00091 0.00091 0.00091"/>
+      <!-- <mesh filename="package://f1tenth-sim/urdf/meshes/chassis.stl" scale="0.000990 0.0009375 0.0009375"/> -->
     </geometry>
   </xacro:macro>
@@ -50,5 +52,5 @@
     <origin xyz="0 0 0" rpy="0 0 0" />
     <geometry>
-      <mesh filename="package://spring_2020_virtual_class/urdf/meshes/left_wheel.stl" />
+      <mesh filename="package://f1tenth-sim/urdf/meshes/left_wheel.stl" />
     </geometry>
   </xacro:macro>
@@ -56,5 +58,5 @@
     <origin xyz="0 0 0" rpy="0 0 0" />
     <geometry>
-      <mesh filename="package://spring_2020_virtual_class/urdf/meshes/right_wheel.stl" />
+      <mesh filename="package://f1tenth-sim/urdf/meshes/right_wheel.stl" />
     </geometry>
   </xacro:macro>
@@ -62,5 +64,5 @@
     <origin xyz="0 0 0" rpy="0 0 0" />
     <geometry>
-      <mesh filename="package://spring_2020_virtual_class/urdf/meshes/left_wheel.stl" />
+      <mesh filename="package://f1tenth-sim/urdf/meshes/left_wheel.stl" />
     </geometry>
   </xacro:macro>
@@ -68,5 +70,5 @@
     <origin xyz="0 0 0" rpy="0 0 0" />
     <geometry>
-      <mesh filename="package://spring_2020_virtual_class/urdf/meshes/right_wheel.stl" />
+      <mesh filename="package://f1tenth-sim/urdf/meshes/right_wheel.stl" />
     </geometry>
   </xacro:macro>
@@ -74,5 +76,5 @@
     <origin xyz="0 0 0" rpy="0 0 0" />
     <geometry>
-      <mesh filename="package://spring_2020_virtual_class/urdf/meshes/hinge.stl" />
+      <mesh filename="package://f1tenth-sim/urdf/meshes/hinge.stl" />
     </geometry>
   </xacro:macro>
@@ -80,5 +82,5 @@
     <origin xyz="0 0 0" rpy="0 0 0" />
     <geometry>
-      <mesh filename="package://spring_2020_virtual_class/urdf/meshes/hinge.stl" />
+      <mesh filename="package://f1tenth-sim/urdf/meshes/hinge.stl" />
     </geometry>
   </xacro:macro>
@@ -127,4 +129,6 @@
       <material name="red" />
     </visual>
+    <collision>
+    </collision>
   </link>
   <joint name="$(arg robot_name)_base_link_joint" type="fixed">
@@ -277,5 +281,5 @@
       <origin xyz="0 0 0" rpy="0 0 0"/>
       <geometry>
-        <mesh filename="package://spring_2020_virtual_class/urdf/meshes/hokuyo.stl"/>
+        <mesh filename="package://f1tenth-sim/urdf/meshes/hokuyo.stl"/>
         <material name="grey" />
       </geometry>

Commit message: realistic behavior updates

File: urdf/macros.xacro (robot description, xacro)
@@ -6,23 +6,36 @@
   <!-- inertial parameter macros -->
   <xacro:macro name="chassis_inertial_params">
-    <origin xyz="0.1477 0 0" rpy="0 0 0" />
-    <mass value="4.0" />
-    <inertia ixx="0.010609" ixy="0"          ixz="0"
+    <!-- <origin xyz="0.1477 0 0" rpy="0 0 0" />
+    <mass value="13.0" /> -->
+    <!-- <inertia ixx="0.010609" ixy="0"          ixz="0"
                             iyy="0.050409"   iyz="0"
-                                             izz="0.05865" />
+                                             izz="0.05865" /> -->
+    <mass value="800.0"/>
+    <origin rpy="0 0 0" xyz="0.1 0 0.4"/>
+    <inertia ixx="140" ixy="0.0" ixz="0.0" iyy="550" iyz="0.0" izz="550"/>
   </xacro:macro>
   <xacro:macro name="left_wheels_inertial_params">
-    <origin xyz="0 0 -0.0225" rpy="0 0 0" />
+    <!-- <origin xyz="0 0 -0.0225" rpy="0 0 0" />
     <mass value="0.34055" />
     <inertia ixx="0.00026046" ixy="0"          ixz="0"
                               iyy="0.00026046" iyz="0"
-                                               izz="0.00041226" />
+                                              izz="0.00041226" /> -->
+    <origin rpy="0 0 0" xyz="0 0 0"/>
+    <mass value="20" />
+    <inertia ixx="0.5" ixy="0"          ixz="0"
+                              iyy="0.5" iyz="0"
+                                               izz="1.0" />
   </xacro:macro>
   <xacro:macro name="right_wheels_inertial_params">
-    <origin xyz="0 0 0.0225" rpy="0 0 0" />
+    <origin rpy="0 0 0" xyz="0 0 0"/>
+    <mass value="20" />
+    <inertia ixx="0.5" ixy="0"          ixz="0"
+                              iyy="0.5" iyz="0"
+                                               izz="1.0" />
+    <!-- <origin xyz="0 0 0.0225" rpy="0 0 0" />
     <mass value="0.34055" />
     <inertia ixx="0.00026046" ixy="0"          ixz="0"
                               iyy="0.00026046" iyz="0"
-                                               izz="0.00041226" />
+                                               izz="0.00041226" /> -->
   </xacro:macro>
   <xacro:macro name="steering_hinge_inertial_params">
@@ -40,10 +53,10 @@
                                                 izz="4E-06" />
   </xacro:macro>
-  <!-- geometry macros -->
+  <!-- visual geometry macros -->
   <xacro:macro name="chassis_geometry">
     <!-- <origin xyz="0.46 -0.135 -0.180" rpy="1.57 0 3.14" /> -->
-    <origin rpy="-1.5708 0 3.1416" xyz="0.175 0.35 0.07"/>
-    <geometry>
-      <mesh filename="package://f1tenth-sim/urdf/meshes/chassis.STL" scale="0.000915 0.000915 0.000915"/>
+    <origin rpy="-1.5708 0 3.1416" xyz="0.165 0.3305 0.0075"/>
+    <geometry>
+      <mesh filename="package://f1tenth-sim/urdf/meshes/chassis.STL" scale="0.00095 0.000925 0.000925"/>
       <!-- <mesh filename="package://f1tenth-sim/urdf/meshes/chassis.stl" scale="0.000990 0.0009375 0.0009375"/> -->
     </geometry>
@@ -85,14 +98,37 @@
     </geometry>
   </xacro:macro>
+  <!-- collision macros -->
   <xacro:macro name="left_wheels_collision_geometry">
     <origin xyz="0 0 -0.0225" rpy="0 0 0" />
     <geometry>
-      <cylinder length="0.045" radius="0.05" />
-    </geometry>
+      <cylinder length="0.062" radius="0.05" />
+    </geometry>
+    <surface>
+      <friction>
+        <ode>
+          <mu>1.0</mu>
+          <mu2>1.0</mu2>
+        </ode>
+      </friction>
+    </surface>
   </xacro:macro>
   <xacro:macro name="right_wheels_collision_geometry">
     <origin xyz="0 0 0.0225" rpy="0 0 0" />
     <geometry>
-      <cylinder length="0.045" radius="0.05" />
+      <cylinder length="0.062" radius="0.05" />
+    </geometry>
+    <surface>
+      <friction>
+        <ode>
+          <mu>1.0</mu>
+          <mu2>1.0</mu2>
+        </ode>
+      </friction>
+    </surface>
+  </xacro:macro>
+  <xacro:macro name="chassis_collision_geometry">
+    <origin xyz="0 0 0.4" rpy="0 0 0" />
+    <geometry>
+      <box size="0.860 0.450 0.180"/>
     </geometry>
   </xacro:macro>
@@ -129,6 +165,7 @@
       <material name="red" />
     </visual>
-    <collision>
-    </collision>
+    <!-- <collision>
+      <xacro:chassis_collision_geometry />
+    </collision> -->
   </link>
   <joint name="$(arg robot_name)_base_link_joint" type="fixed">
@@ -287,5 +324,5 @@
   </link>
   <joint name="$(arg robot_name)_hokuyo_joint" type="fixed">
-    <origin xyz="0.125 0.0 0.155" rpy="0 0 0"/>
+    <origin xyz="0.35 0.0 0.075" rpy="0 0 0"/>
     <parent link="$(arg robot_name)_chassis" />
     <child link="$(arg robot_name)_laser" />

Commit message: revisions for look

File: urdf/macros.xacro (robot description, xacro)
@@ -4,38 +4,39 @@
   <xacro:arg name="robot_name" default="car_1" />
   <xacro:arg name="robot_skin" default="Blue" />
+<!-- ###### INERTIA, VISUAL, & COLLISION MACROS ####################################-->
   <!-- inertial parameter macros -->
   <xacro:macro name="chassis_inertial_params">
-    <!-- <origin xyz="0.1477 0 0" rpy="0 0 0" />
-    <mass value="13.0" /> -->
-    <!-- <inertia ixx="0.010609" ixy="0"          ixz="0"
+    <origin xyz="0.1477 0 0" rpy="0 0 0" />
+    <mass value="13.0" />
+    <inertia ixx="0.010609" ixy="0"          ixz="0"
                             iyy="0.050409"   iyz="0"
-                                             izz="0.05865" /> -->
-    <mass value="800.0"/>
-    <origin rpy="0 0 0" xyz="0.1 0 0.4"/>
-    <inertia ixx="140" ixy="0.0" ixz="0.0" iyy="550" iyz="0.0" izz="550"/>
+                                             izz="0.05865" />
+    <!-- <mass value="800.0"/>
+    <origin rpy="0 0 0" xyz="0.1477 0 0"/>
+    <inertia ixx="140" ixy="0.0" ixz="0.0" iyy="550" iyz="0.0" izz="550"/> -->
   </xacro:macro>
   <xacro:macro name="left_wheels_inertial_params">
-    <!-- <origin xyz="0 0 -0.0225" rpy="0 0 0" />
-    <mass value="0.34055" />
+    <origin xyz="0 0 -0.0225" rpy="0 0 0" />
+    <mass value="0.453592" />
     <inertia ixx="0.00026046" ixy="0"          ixz="0"
                               iyy="0.00026046" iyz="0"
-                                              izz="0.00041226" /> -->
-    <origin rpy="0 0 0" xyz="0 0 0"/>
+                                              izz="0.00041226" />
+    <!-- <origin rpy="0 0 0" xyz="0 0 0"/>
     <mass value="20" />
     <inertia ixx="0.5" ixy="0"          ixz="0"
                               iyy="0.5" iyz="0"
-                                               izz="1.0" />
+                                               izz="1.0" /> -->
   </xacro:macro>
   <xacro:macro name="right_wheels_inertial_params">
-    <origin rpy="0 0 0" xyz="0 0 0"/>
+    <!-- <origin rpy="0 0 0" xyz="0 0 0"/>
     <mass value="20" />
     <inertia ixx="0.5" ixy="0"          ixz="0"
                               iyy="0.5" iyz="0"
-                                               izz="1.0" />
-    <!-- <origin xyz="0 0 0.0225" rpy="0 0 0" />
-    <mass value="0.34055" />
+                                               izz="1.0" /> -->
+    <origin xyz="0 0 0.0225" rpy="0 0 0" />
+    <mass value="0.453592" />
     <inertia ixx="0.00026046" ixy="0"          ixz="0"
                               iyy="0.00026046" iyz="0"
-                                               izz="0.00041226" /> -->
+                                               izz="0.00041226" />
   </xacro:macro>
   <xacro:macro name="steering_hinge_inertial_params">
@@ -56,5 +57,5 @@
   <xacro:macro name="chassis_geometry">
     <!-- <origin xyz="0.46 -0.135 -0.180" rpy="1.57 0 3.14" /> -->
-    <origin rpy="-1.5708 0 3.1416" xyz="0.165 0.3305 0.0075"/>
+    <origin rpy="-1.5708 0 3.1416" xyz="0.165 0.3305 -0.01"/>
     <geometry>
       <mesh filename="package://f1tenth-sim/urdf/meshes/chassis.STL" scale="0.00095 0.000925 0.000925"/>
@@ -63,25 +64,29 @@
   </xacro:macro>
   <xacro:macro name="left_rear_wheel_geometry">
-    <origin xyz="0 0 0" rpy="0 0 0" />
-    <geometry>
-      <mesh filename="package://f1tenth-sim/urdf/meshes/left_wheel.stl" />
+    <origin xyz="0 0 0.0225" rpy="0 0 0" />
+    <geometry>
+      <!-- <mesh filename="package://f1tenth-sim/urdf/meshes/left_wheel.stl" /> -->
+      <mesh filename="package://f1tenth-sim/urdf/meshes/wheel.dae" scale="0.0012 0.0012 0.0012"/>
     </geometry>
   </xacro:macro>
   <xacro:macro name="right_rear_wheel_geometry">
-    <origin xyz="0 0 0" rpy="0 0 0" />
-    <geometry>
-      <mesh filename="package://f1tenth-sim/urdf/meshes/right_wheel.stl" />
+    <origin xyz="0 0 0.0225" rpy="0 0 0" />
+    <geometry>
+      <!-- <mesh filename="package://f1tenth-sim/urdf/meshes/right_wheel.stl" /> -->
+      <mesh filename="package://f1tenth-sim/urdf/meshes/wheel.dae" scale="0.0012 0.0012 0.0012"/>
     </geometry>
   </xacro:macro>
   <xacro:macro name="left_front_wheel_geometry">
-    <origin xyz="0 0 0" rpy="0 0 0" />
-    <geometry>
-      <mesh filename="package://f1tenth-sim/urdf/meshes/left_wheel.stl" />
+    <origin xyz="0 0 0.0225" rpy="0 0 0" />
+    <geometry>
+      <!-- <mesh filename="package://f1tenth-sim/urdf/meshes/left_wheel.stl" /> -->
+      <mesh filename="package://f1tenth-sim/urdf/meshes/wheel.dae" scale="0.0012 0.0012 0.0012"/>
     </geometry>
   </xacro:macro>
   <xacro:macro name="right_front_wheel_geometry">
-    <origin xyz="0 0 0" rpy="0 0 0" />
-    <geometry>
-      <mesh filename="package://f1tenth-sim/urdf/meshes/right_wheel.stl" />
+    <origin xyz="0 0 0.0225" rpy="0 0 0" />
+    <geometry>
+      <!-- <mesh filename="package://f1tenth-sim/urdf/meshes/right_wheel.stl" /> -->
+      <mesh filename="package://f1tenth-sim/urdf/meshes/wheel.dae" scale="0.0012 0.0012 0.0012"/>
     </geometry>
   </xacro:macro>
@@ -100,9 +105,9 @@
   <!-- collision macros -->
   <xacro:macro name="left_wheels_collision_geometry">
-    <origin xyz="0 0 -0.0225" rpy="0 0 0" />
-    <geometry>
-      <cylinder length="0.062" radius="0.05" />
-    </geometry>
-    <surface>
+    <origin xyz="0 0 0.0225" rpy="0 0 0" />
+    <geometry>
+      <cylinder length="0.055" radius="0.06" />
+    </geometry>
+    <!-- <surface>
       <friction>
         <ode>
@@ -111,12 +116,12 @@
         </ode>
       </friction>
-    </surface>
+    </surface> -->
   </xacro:macro>
   <xacro:macro name="right_wheels_collision_geometry">
     <origin xyz="0 0 0.0225" rpy="0 0 0" />
     <geometry>
-      <cylinder length="0.062" radius="0.05" />
-    </geometry>
-    <surface>
+      <cylinder length="0.055" radius="0.06" />
+    </geometry>
+    <!-- <surface>
       <friction>
         <ode>
@@ -125,5 +130,5 @@
         </ode>
       </friction>
-    </surface>
+    </surface> -->
   </xacro:macro>
   <xacro:macro name="chassis_collision_geometry">
@@ -158,4 +163,5 @@
     </transmission>
   </xacro:macro>
+<!-- ###### LINK & JOINT DEFINTIONS ####################################-->
   <!-- Add chassis and it's inertia link -->
   <link name="$(arg robot_name)_base_link"/>
@@ -184,4 +190,25 @@
     <child link="$(arg robot_name)_chassis_inertia" />
   </joint>
+  <!-- Add the left front wheel with its joints and tranmissions -->
+  <link name="$(arg robot_name)_left_front_wheel">
+    <inertial>
+      <xacro:left_wheels_inertial_params />
+    </inertial>
+    <visual>
+      <xacro:left_front_wheel_geometry />
+      <material name="black" />
+    </visual>
+    <collision>
+      <xacro:left_wheels_collision_geometry />
+    </collision>
+  </link>
+  <joint name="$(arg robot_name)_left_front_wheel_joint" type="continuous">
+    <origin xyz="0 0 0" rpy="-1.5708 0 0" />
+    <parent link="$(arg robot_name)_left_steering_hinge" />
+    <child link="$(arg robot_name)_left_front_wheel" />
+    <axis xyz="0 0 -1" />
+    <limit effort="10" velocity="100" />
+  </joint>
+  <xacro:wheel_transmission name="$(arg robot_name)_left_front_wheel" />
   <!-- Add the left rear wheel with its joints and tranmissions -->
   <link name="$(arg robot_name)_left_rear_wheel">
@@ -198,5 +225,5 @@
   </link>
   <joint name="$(arg robot_name)_left_rear_wheel_joint" type="continuous">
-    <origin xyz="0 0.1 0" rpy="1.5708 0 0" />
+    <origin xyz="0 0.1 0" rpy="-1.5708 0 0" />
     <parent link="$(arg robot_name)_chassis" />
     <child link="$(arg robot_name)_left_rear_wheel" />
@@ -205,4 +232,25 @@
   </joint>
   <xacro:wheel_transmission name="$(arg robot_name)_left_rear_wheel" />
+  <!-- Add the right front wheel with its joints and tranmissions -->
+  <link name="$(arg robot_name)_right_front_wheel">
+    <inertial>
+      <xacro:right_wheels_inertial_params />
+    </inertial>
+    <visual>
+      <xacro:right_front_wheel_geometry />
+      <material name="black" />
+    </visual>
+    <collision>
+      <xacro:right_wheels_collision_geometry />
+    </collision>
+  </link>
+  <joint name="$(arg robot_name)_right_front_wheel_joint" type="continuous">
+    <origin xyz="0 0 0" rpy="1.5708 0 0" />
+    <parent link="$(arg robot_name)_right_steering_hinge" />
+    <child link="$(arg robot_name)_right_front_wheel" />
+    <axis xyz="0 0 -1" />
+    <limit effort="10" velocity="100"/>
+  </joint>
+  <xacro:wheel_transmission name="$(arg robot_name)_right_front_wheel" />
   <!-- Add the right rear wheel with its joints and tranmissions -->
   <link name="$(arg robot_name)_right_rear_wheel">
@@ -212,5 +260,5 @@
     <visual>
       <xacro:right_rear_wheel_geometry />
-      <material name="black" />
+      <material name="red" />
     </visual>
     <collision>
@@ -237,9 +285,9 @@
   </link>
   <joint name="$(arg robot_name)_left_steering_hinge_joint" type="revolute">
-    <origin xyz="0.325 0.1 0" rpy="0 1.5708 0" />
+    <origin xyz="0.325 0.1 0" rpy="0 0 0" />
     <parent link="$(arg robot_name)_chassis" />
     <child link="$(arg robot_name)_left_steering_hinge" />
-    <axis xyz="-1 0 0" />
-    <limit lower="-1.0" upper="1.0" effort="10" velocity="100" />
+    <axis xyz="0 0 1" />
+    <limit lower="-0.523599" upper="0.523599" effort="10" velocity="100" />
   </joint>
   <xacro:steering_hinge_transmission name="$(arg robot_name)_left_steering_hinge" />
@@ -254,54 +302,12 @@
     </visual>
   </link>
-  <joint name="$(arg robot_name)_right_steering_hinge_joint" type="continuous">
-    <origin xyz="0.325 -0.1 0" rpy="0 1.5708 0" />
+  <joint name="$(arg robot_name)_right_steering_hinge_joint" type="revolute">
+    <origin xyz="0.325 -0.1 0" rpy="0 0 0" />
     <parent link="$(arg robot_name)_chassis" />
     <child link="$(arg robot_name)_right_steering_hinge" />
-    <axis xyz="-1 0 0" />
-    <limit lower="-1.0" upper="1.0" effort="10" velocity="100" />
+    <axis xyz="0 0 1" />
+    <limit lower="-0.523599" upper="0.523599" effort="10" velocity="100" />
   </joint>
   <xacro:steering_hinge_transmission name="$(arg robot_name)_right_steering_hinge" />
-  <!-- Add the left front wheel with its joints and tranmissions -->
-  <link name="$(arg robot_name)_left_front_wheel">
-    <inertial>
-      <xacro:left_wheels_inertial_params />
-    </inertial>
-    <visual>
-      <xacro:left_front_wheel_geometry />
-      <material name="black" />
-    </visual>
-    <collision>
-      <xacro:left_wheels_collision_geometry />
-    </collision>
-  </link>
-  <joint name="$(arg robot_name)_left_front_wheel_joint" type="continuous">
-    <origin xyz="0 0 0" rpy="1.5708 0 0" />
-    <parent link="$(arg robot_name)_left_steering_hinge" />
-    <child link="$(arg robot_name)_left_front_wheel" />
-    <axis xyz="0 0 -1" />
-    <limit effort="10" velocity="100" />
-  </joint>
-  <xacro:wheel_transmission name="$(arg robot_name)_left_front_wheel" />
-  <!-- Add the left front wheel with its joints and tranmissions -->
-  <link name="$(arg robot_name)_right_front_wheel">
-    <inertial>
-      <xacro:right_wheels_inertial_params />
-    </inertial>
-    <visual>
-      <xacro:right_front_wheel_geometry />
-      <material name="black" />
-    </visual>
-    <collision>
-      <xacro:right_wheels_collision_geometry />
-    </collision>
-  </link>
-  <joint name="$(arg robot_name)_right_front_wheel_joint" type="continuous">
-    <origin xyz="0 0 0" rpy="1.5708 0 0" />
-    <parent link="$(arg robot_name)_right_steering_hinge" />
-    <child link="$(arg robot_name)_right_front_wheel" />
-    <axis xyz="0 0 -1" />
-    <limit effort="10" velocity="100"/>
-  </joint>
-  <xacro:wheel_transmission name="$(arg robot_name)_right_front_wheel" />
   <!-- Add Hokuyo laser scanner -->
   <link name="$(arg robot_name)_laser">
@@ -384,5 +390,6 @@
     <axis xyz="0 0 1" />
   </joint>
-  <!-- Gazebo references -->
+<!-- #### GAZEBO SIMULATION SETTINGS #### -->
+  <!-- Gazebo Material References -->
   <gazebo reference="$(arg robot_name)_chassis">
     <mu1 value="0.0"/>
@@ -398,5 +405,5 @@
     <kd  value="1.0" />
     <fdir1 value="1 0 0"/>
-    <material>Gazebo/Black</material>
+    <material>Gazebo/DarkGrey</material>
   </gazebo>
   <gazebo reference="$(arg robot_name)_right_rear_wheel">
@@ -406,5 +413,5 @@
     <kd  value="1.0" />
     <fdir1 value="1 0 0"/>
-    <material>Gazebo/Black</material>
+    <material>Gazebo/DarkGrey</material>
   </gazebo>
   <gazebo reference="$(arg robot_name)_left_front_wheel">
@@ -414,5 +421,5 @@
     <kd  value="1.0" />
     <fdir1 value="0 0 1"/>
-    <material>Gazebo/Black</material>
+    <material>Gazebo/DarkGrey</material>
   </gazebo>
   <gazebo reference="$(arg robot_name)_right_front_wheel">
@@ -422,5 +429,5 @@
     <kd  value="1.0" />
     <fdir1 value="0 0 1"/>
-    <material>Gazebo/Black</material>
+    <material>Gazebo/DarkGrey</material>
   </gazebo>
   <!-- Gazebo plugins -->
