Commit message: direct angular velocity setpoints

File: urdf/macros.xacro (robot description, xacro)
@@ -60,5 +60,4 @@
     <geometry>
       <mesh filename="package://f1tenth-sim/urdf/meshes/chassis.STL" scale="0.00095 0.000925 0.000925"/>
-      <!-- <mesh filename="package://f1tenth-sim/urdf/meshes/chassis.stl" scale="0.000990 0.0009375 0.0009375"/> -->
     </geometry>
   </xacro:macro>
@@ -66,5 +65,4 @@
     <origin xyz="0 0 0.0225" rpy="0 0 0" />
     <geometry>
-      <!-- <mesh filename="package://f1tenth-sim/urdf/meshes/left_wheel.stl" /> -->
       <mesh filename="package://f1tenth-sim/urdf/meshes/wheel.dae" scale="0.0012 0.0012 0.0012"/>
     </geometry>
@@ -73,5 +71,4 @@
     <origin xyz="0 0 0.0225" rpy="0 0 0" />
     <geometry>
-      <!-- <mesh filename="package://f1tenth-sim/urdf/meshes/right_wheel.stl" /> -->
       <mesh filename="package://f1tenth-sim/urdf/meshes/wheel.dae" scale="0.0012 0.0012 0.0012"/>
     </geometry>
@@ -80,5 +77,4 @@
     <origin xyz="0 0 0.0225" rpy="0 0 0" />
     <geometry>
-      <!-- <mesh filename="package://f1tenth-sim/urdf/meshes/left_wheel.stl" /> -->
       <mesh filename="package://f1tenth-sim/urdf/meshes/wheel.dae" scale="0.0012 0.0012 0.0012"/>
     </geometry>
@@ -87,5 +83,4 @@
     <origin xyz="0 0 0.0225" rpy="0 0 0" />
     <geometry>
-      <!-- <mesh filename="package://f1tenth-sim/urdf/meshes/right_wheel.stl" /> -->
       <mesh filename="package://f1tenth-sim/urdf/meshes/wheel.dae" scale="0.0012 0.0012 0.0012"/>
     </geometry>
@@ -104,4 +99,10 @@
   </xacro:macro>
   <!-- collision macros -->
+  <xacro:macro name="chassis_collision_geometry">
+    <origin xyz="0 0 -0.3" rpy="0 0 0" />
+    <geometry>
+      <box size="0.860 0.450 0.001"/>
+    </geometry>
+  </xacro:macro>
   <xacro:macro name="left_wheels_collision_geometry">
     <origin xyz="0 0 0.0225" rpy="0 0 0" />
@@ -131,10 +132,4 @@
       </friction>
     </surface> -->
-  </xacro:macro>
-  <xacro:macro name="chassis_collision_geometry">
-    <origin xyz="0 0 0.4" rpy="0 0 0" />
-    <geometry>
-      <box size="0.860 0.450 0.180"/>
-    </geometry>
   </xacro:macro>
   <!-- transmission macros -->
@@ -207,5 +202,5 @@
     <parent link="$(arg robot_name)_left_steering_hinge" />
     <child link="$(arg robot_name)_left_front_wheel" />
-    <axis xyz="0 0 -1" />
+    <axis xyz="0 0 1" />
     <limit effort="10" velocity="100" />
   </joint>
@@ -228,5 +223,5 @@
     <parent link="$(arg robot_name)_chassis" />
     <child link="$(arg robot_name)_left_rear_wheel" />
-    <axis xyz="0 0 -1" />
+    <axis xyz="0 0 1" />
     <limit effort="10" velocity="100" />
   </joint>
@@ -335,5 +330,5 @@
     <axis xyz="0 0 1" />
   </joint>
-  <!-- camera class (spawn parameters) -->
+  camera class (spawn parameters)
   <link name="$(arg robot_name)_link">
     <inertial>

Commit message: migration

File: urdf/macros.xacro (robot description, xacro)
@@ -12,26 +12,13 @@
                             iyy="0.050409"   iyz="0"
                                              izz="0.05865" />
-    <!-- <mass value="800.0"/>
-    <origin rpy="0 0 0" xyz="0.1477 0 0"/>
-    <inertia ixx="140" ixy="0.0" ixz="0.0" iyy="550" iyz="0.0" izz="550"/> -->
   </xacro:macro>
   <xacro:macro name="left_wheels_inertial_params">
-    <origin xyz="0 0 -0.0225" rpy="0 0 0" />
+    <origin xyz="0 0 0.0225" rpy="0 0 0" />
     <mass value="0.453592" />
     <inertia ixx="0.00026046" ixy="0"          ixz="0"
                               iyy="0.00026046" iyz="0"
                                               izz="0.00041226" />
-    <!-- <origin rpy="0 0 0" xyz="0 0 0"/>
-    <mass value="20" />
-    <inertia ixx="0.5" ixy="0"          ixz="0"
-                              iyy="0.5" iyz="0"
-                                               izz="1.0" /> -->
   </xacro:macro>
   <xacro:macro name="right_wheels_inertial_params">
-    <!-- <origin rpy="0 0 0" xyz="0 0 0"/>
-    <mass value="20" />
-    <inertia ixx="0.5" ixy="0"          ixz="0"
-                              iyy="0.5" iyz="0"
-                                               izz="1.0" /> -->
     <origin xyz="0 0 0.0225" rpy="0 0 0" />
     <mass value="0.453592" />
@@ -185,5 +172,5 @@
     <child link="$(arg robot_name)_chassis_inertia" />
   </joint>
-  <!-- Add the left front wheel with its joints and tranmissions -->
+  <!-- Add the left front wheel with its joints and transmissions -->
   <link name="$(arg robot_name)_left_front_wheel">
     <inertial>
@@ -203,8 +190,8 @@
     <child link="$(arg robot_name)_left_front_wheel" />
     <axis xyz="0 0 1" />
-    <limit effort="10" velocity="100" />
+    <limit effort="20" velocity="300" />
   </joint>
   <xacro:wheel_transmission name="$(arg robot_name)_left_front_wheel" />
-  <!-- Add the left rear wheel with its joints and tranmissions -->
+  <!-- Add the left rear wheel with its joints and transmissions -->
   <link name="$(arg robot_name)_left_rear_wheel">
     <inertial>
@@ -224,8 +211,8 @@
     <child link="$(arg robot_name)_left_rear_wheel" />
     <axis xyz="0 0 1" />
-    <limit effort="10" velocity="100" />
+    <limit effort="20" velocity="300" />
   </joint>
   <xacro:wheel_transmission name="$(arg robot_name)_left_rear_wheel" />
-  <!-- Add the right front wheel with its joints and tranmissions -->
+  <!-- Add the right front wheel with its joints and transmissions -->
   <link name="$(arg robot_name)_right_front_wheel">
     <inertial>
@@ -245,8 +232,8 @@
     <child link="$(arg robot_name)_right_front_wheel" />
     <axis xyz="0 0 -1" />
-    <limit effort="10" velocity="100"/>
+    <limit effort="20" velocity="300" />
   </joint>
   <xacro:wheel_transmission name="$(arg robot_name)_right_front_wheel" />
-  <!-- Add the right rear wheel with its joints and tranmissions -->
+  <!-- Add the right rear wheel with its joints and transmissions -->
   <link name="$(arg robot_name)_right_rear_wheel">
     <inertial>
@@ -266,8 +253,8 @@
     <child link="$(arg robot_name)_right_rear_wheel" />
     <axis xyz="0 0 -1" />
-    <limit effort="10" velocity="100" />
+    <limit effort="20" velocity="300" />
   </joint>
   <xacro:wheel_transmission name="$(arg robot_name)_right_rear_wheel" />
-  <!-- Add the left steering hinge with its joints and tranmissions -->
+  <!-- Add the left steering hinge with its joints and transmissions -->
   <link name="$(arg robot_name)_left_steering_hinge">
     <inertial>
@@ -287,5 +274,5 @@
   </joint>
   <xacro:steering_hinge_transmission name="$(arg robot_name)_left_steering_hinge" />
-  <!-- Add the right steering hinge with its joints and tranmissions -->
+  <!-- Add the right steering hinge with its joints and transmissions -->
   <link name="$(arg robot_name)_right_steering_hinge">
     <inertial>
@@ -313,5 +300,5 @@
       <origin xyz="0 0 0" rpy="0 0 0"/>
       <geometry>
-        <box size="0.1 0.1 0.1"/>
+        <box size="0.060 0.060 0.080"/>
       </geometry>
     </collision>
@@ -330,6 +317,6 @@
     <axis xyz="0 0 1" />
   </joint>
-  camera class (spawn parameters)
-  <link name="$(arg robot_name)_link">
+  <!-- camera class (spawn parameters) -->
+  <!-- <link name="$(arg robot_name)_link">
     <inertial>
       <mass value="1e-5" />
@@ -356,8 +343,7 @@
     <child link="$(arg robot_name)_link"/>
     <axis xyz="0 0 1" />
-    <!-- <limit lower="0.0" upper="0.0" effort="0.0" velocity="0.0" /> -->
-  </joint>
+  </joint> -->
   <!-- camera lenses -->
-  <link name="$(arg robot_name)_camera_link">
+  <!-- <link name="$(arg robot_name)_camera_link">
     <inertial>
       <mass value="1e-5" />
@@ -384,10 +370,10 @@
     <child link="$(arg robot_name)_right_link"/>
     <axis xyz="0 0 1" />
-  </joint>
+  </joint> -->
 <!-- #### GAZEBO SIMULATION SETTINGS #### -->
   <!-- Gazebo Material References -->
   <gazebo reference="$(arg robot_name)_chassis">
-    <mu1 value="0.0"/>
-    <mu2 value="0.0"/>
+    <mu1 value="0.0"/>                  <!-- should be the same as the material contacting it -->
+    <mu2 value="0.0"/>                  <!-- should be the same as the material contacting it -->
     <kp  value="10000000.0" />
     <kd  value="1.0" />
@@ -415,5 +401,6 @@
     <kp  value="10000000.0" />
     <kd  value="1.0" />
-    <fdir1 value="0 0 1"/>
+    <!-- <fdir1 value="0 0 1"/> -->
+    <fdir1 value="1 0 0"/>
     <material>Gazebo/DarkGrey</material>
   </gazebo>
@@ -423,5 +410,6 @@
     <kp  value="10000000.0" />
     <kd  value="1.0" />
-    <fdir1 value="0 0 1"/>
+    <!-- <fdir1 value="0 0 1"/> -->
+    <fdir1 value="1 0 0"/>
     <material>Gazebo/DarkGrey</material>
   </gazebo>
@@ -446,5 +434,5 @@
     </plugin>
   </gazebo>
-    <!-- hokuyo -->
+  <!-- hokuyo -->
   <xacro:unless value="$(optenv DISABLE_GAZEBO_LASER false)">
     <gazebo reference="$(arg robot_name)_laser">

Commit message: sim ready

File: urdf/macros.xacro (robot description, xacro)
@@ -4,4 +4,10 @@
   <xacro:arg name="robot_name" default="car_1" />
   <xacro:arg name="robot_skin" default="Blue" />
+  <xacro:property name="WHEELSURFACEFRICTION" value="0.9" />
+  <xacro:property name="WHEELSURFACESLIP" value="0.1" />
+  <xacro:property name="WHEELJOINTDAMPING" value="0.5" />
+  <xacro:property name="WHEELJOINTFRICTION" value="0.5" />
+  <xacro:property name="WHEEL_WIDTH" value="0.06" />
+  <xacro:property name="WHEEL_RADIUS" value="0.055" />
 <!-- ###### INERTIA, VISUAL, & COLLISION MACROS ####################################-->
   <!-- inertial parameter macros -->
@@ -43,5 +49,4 @@
   <!-- visual geometry macros -->
   <xacro:macro name="chassis_geometry">
-    <!-- <origin xyz="0.46 -0.135 -0.180" rpy="1.57 0 3.14" /> -->
     <origin rpy="-1.5708 0 3.1416" xyz="0.165 0.3305 -0.01"/>
     <geometry>
@@ -95,28 +100,12 @@
     <origin xyz="0 0 0.0225" rpy="0 0 0" />
     <geometry>
-      <cylinder length="0.055" radius="0.06" />
-    </geometry>
-    <!-- <surface>
-      <friction>
-        <ode>
-          <mu>1.0</mu>
-          <mu2>1.0</mu2>
-        </ode>
-      </friction>
-    </surface> -->
+      <cylinder length="${WHEEL_WIDTH}" radius="${WHEEL_RADIUS}" />
+    </geometry>
   </xacro:macro>
   <xacro:macro name="right_wheels_collision_geometry">
     <origin xyz="0 0 0.0225" rpy="0 0 0" />
     <geometry>
-      <cylinder length="0.055" radius="0.06" />
-    </geometry>
-    <!-- <surface>
-      <friction>
-        <ode>
-          <mu>1.0</mu>
-          <mu2>1.0</mu2>
-        </ode>
-      </friction>
-    </surface> -->
+      <cylinder length="${WHEEL_WIDTH}" radius="${WHEEL_RADIUS}" />
+    </geometry>
   </xacro:macro>
   <!-- transmission macros -->
@@ -155,5 +144,15 @@
     <!-- <collision>
       <xacro:chassis_collision_geometry />
-    </collision> -->
+    </collision>
+    <surface>
+        <friction>
+            <ode>
+                <mu>${WHEELSURFACEFRICTION}</mu>
+                <mu2>${WHEELSURFACEFRICTION}</mu2>
+                <slip1>${WHEELSURFACESLIP}</slip1>
+                <slip2>${WHEELSURFACESLIP}</slip2>
+            </ode>
+        </friction>
+    </surface> -->
   </link>
   <joint name="$(arg robot_name)_base_link_joint" type="fixed">
@@ -184,4 +183,14 @@
       <xacro:left_wheels_collision_geometry />
     </collision>
+    <surface>
+        <friction>
+            <ode>
+                <mu>${WHEELSURFACEFRICTION}</mu>
+                <mu2>${WHEELSURFACEFRICTION}</mu2>
+                <slip1>${WHEELSURFACESLIP}</slip1>
+                <slip2>${WHEELSURFACESLIP}</slip2>
+            </ode>
+        </friction>
+    </surface>
   </link>
   <joint name="$(arg robot_name)_left_front_wheel_joint" type="continuous">
@@ -190,4 +199,5 @@
     <child link="$(arg robot_name)_left_front_wheel" />
     <axis xyz="0 0 1" />
+    <joint_properties damping="${WHEELJOINTDAMPING}" friction="${WHEELJOINTFRICTION}"/>
     <limit effort="20" velocity="300" />
   </joint>
@@ -205,4 +215,14 @@
       <xacro:left_wheels_collision_geometry />
     </collision>
+    <surface>
+        <friction>
+            <ode>
+                <mu>${WHEELSURFACEFRICTION}</mu>
+                <mu2>${WHEELSURFACEFRICTION}</mu2>
+                <slip1>${WHEELSURFACESLIP}</slip1>
+                <slip2>${WHEELSURFACESLIP}</slip2>
+            </ode>
+        </friction>
+    </surface>
   </link>
   <joint name="$(arg robot_name)_left_rear_wheel_joint" type="continuous">
@@ -226,4 +246,14 @@
       <xacro:right_wheels_collision_geometry />
     </collision>
+    <surface>
+        <friction>
+            <ode>
+                <mu>${WHEELSURFACEFRICTION}</mu>
+                <mu2>${WHEELSURFACEFRICTION}</mu2>
+                <slip1>${WHEELSURFACESLIP}</slip1>
+                <slip2>${WHEELSURFACESLIP}</slip2>
+            </ode>
+        </friction>
+    </surface>
   </link>
   <joint name="$(arg robot_name)_right_front_wheel_joint" type="continuous">
@@ -247,4 +277,14 @@
       <xacro:right_wheels_collision_geometry />
     </collision>
+    <surface>
+        <friction>
+            <ode>
+                <mu>${WHEELSURFACEFRICTION}</mu>
+                <mu2>${WHEELSURFACEFRICTION}</mu2>
+                <slip1>${WHEELSURFACESLIP}</slip1>
+                <slip2>${WHEELSURFACESLIP}</slip2>
+            </ode>
+        </friction>
+    </surface>
   </link>
   <joint name="$(arg robot_name)_right_rear_wheel_joint" type="continuous">
@@ -374,6 +414,4 @@
   <!-- Gazebo Material References -->
   <gazebo reference="$(arg robot_name)_chassis">
-    <mu1 value="0.0"/>                  <!-- should be the same as the material contacting it -->
-    <mu2 value="0.0"/>                  <!-- should be the same as the material contacting it -->
     <kp  value="10000000.0" />
     <kd  value="1.0" />
@@ -381,35 +419,21 @@
   </gazebo>
   <gazebo reference="$(arg robot_name)_left_rear_wheel">
-    <mu1 value="1.0"/>
-    <mu2 value="1.0"/>
     <kp  value="10000000.0" />
     <kd  value="1.0" />
-    <fdir1 value="1 0 0"/>
     <material>Gazebo/DarkGrey</material>
   </gazebo>
   <gazebo reference="$(arg robot_name)_right_rear_wheel">
-    <mu1 value="1.0"/>
-    <mu2 value="1.0"/>
     <kp  value="10000000.0" />
     <kd  value="1.0" />
-    <fdir1 value="1 0 0"/>
     <material>Gazebo/DarkGrey</material>
   </gazebo>
   <gazebo reference="$(arg robot_name)_left_front_wheel">
-    <mu1 value="1.0"/>
-    <mu2 value="1.0"/>
     <kp  value="10000000.0" />
     <kd  value="1.0" />
-    <!-- <fdir1 value="0 0 1"/> -->
-    <fdir1 value="1 0 0"/>
     <material>Gazebo/DarkGrey</material>
   </gazebo>
   <gazebo reference="$(arg robot_name)_right_front_wheel">
-    <mu1 value="1.0"/>
-    <mu2 value="1.0"/>
     <kp  value="10000000.0" />
     <kd  value="1.0" />
-    <!-- <fdir1 value="0 0 1"/> -->
-    <fdir1 value="1 0 0"/>
     <material>Gazebo/DarkGrey</material>
   </gazebo>
